Commit message: fixed description

File: src/dh_ag95_description/urdf/dh_ag95.ros2_control.xacro (robot description, xacro)
@@ -1,11 +1,22 @@
 <?xml version="1.0"?>
 <robot xmlns:xacro="http://www.ros.org/wiki/xacro">
-  <!-- Pure ros2_control definition macro, no visual/collision geometry. -->
-  <xacro:macro name="dh_ag95_ros2_control" params="name:=dh_ag95 prefix:=dh_ag95 gripper_id:=1 transport_type:=official_serial port:=/dev/ttyACM0 baudrate:=115200 can_interface:=can0 can_bitrate:=500000 pcan_channel:=PCAN_USBBUS1 pcan_bitrate:=500000 command_unit:=normalized auto_initialize:=true default_force_percent:=30">
-    <ros2_control name="${name}_hardware" type="actuator">
+  <xacro:macro name="dh_ag95_ros2_control" params="
+      name:=dh_ag95_hardware
+      prefix:=
+      transport_type:=official_serial
+      port:=/dev/ttyACM0
+      baudrate:=115200
+      can_interface:=can0
+      can_bitrate:=500000
+      pcan_channel:=PCAN_USBBUS1
+      pcan_bitrate:=500000
+      gripper_id:=1
+      command_unit:=normalized
+      stroke_m:=0.095
+      default_force_percent:=30
+      auto_initialize:=true">
+    <ros2_control name="${name}" type="actuator">
       <hardware>
         <plugin>dh_ag95_controllers/DhAg95Hardware</plugin>
-        <param name="joint_name">${prefix}_finger_joint</param>
-        <param name="gripper_id">${gripper_id}</param>
         <param name="transport_type">${transport_type}</param>
         <param name="port">${port}</param>
@@ -15,16 +26,19 @@
         <param name="pcan_channel">${pcan_channel}</param>
         <param name="pcan_bitrate">${pcan_bitrate}</param>
-        <param name="command_interval_ms">30</param>
-        <param name="read_timeout_ms">200</param>
+        <param name="gripper_id">${gripper_id}</param>
+        <param name="command_unit">${command_unit}</param>
+        <param name="stroke_m">${stroke_m}</param>
+        <param name="default_force_percent">${default_force_percent}</param>
         <param name="auto_initialize">${auto_initialize}</param>
-        <param name="default_force_percent">${default_force_percent}</param>
-        <param name="command_unit">${command_unit}</param>
-        <param name="stroke_m">0.095</param>
-        <param name="invert_position">false</param>
-        <param name="write_deadband">0.01</param>
       </hardware>
-      <joint name="${prefix}_finger_joint">
-        <command_interface name="position"/>
-        <command_interface name="effort"/>
+      <joint name="${prefix}gripper_finger1_joint">
+        <command_interface name="position">
+          <param name="min">0.0</param>
+          <param name="max">1.0</param>
+        </command_interface>
+        <command_interface name="effort">
+          <param name="min">20.0</param>
+          <param name="max">100.0</param>
+        </command_interface>
         <state_interface name="position"/>
         <state_interface name="velocity"/>

File: src/dh_ag95_description/urdf/dh_ag95.urdf.xacro (robot description, xacro)
@@ -1,8 +1,14 @@
 <?xml version="1.0"?>
 <robot name="dh_ag95" xmlns:xacro="http://www.ros.org/wiki/xacro">
-  <xacro:arg name="prefix" default="dh_ag95"/>
+  <xacro:arg name="prefix" default=""/>
+  <xacro:include filename="$(find dh_ag95_description)/urdf/dh_ag95_macro.urdf.xacro"/>
   <link name="world"/>
-  <xacro:include filename="$(find dh_ag95_description)/urdf/dh_ag95_macro.urdf.xacro"/>
-  <xacro:dh_ag95_gripper prefix="$(arg prefix)" parent="world">
+  <link name="$(arg prefix)ag95_mount_link"/>
+  <joint name="$(arg prefix)world_to_ag95_mount" type="fixed">
+    <parent link="world"/>
+    <child link="$(arg prefix)ag95_mount_link"/>
+    <origin xyz="0 0 0" rpy="0 0 0"/>
+  </joint>
+  <xacro:dh_ag95_gripper prefix="$(arg prefix)" parent="$(arg prefix)ag95_mount_link">
     <origin xyz="0 0 0" rpy="0 0 0"/>
   </xacro:dh_ag95_gripper>

File: src/dh_ag95_description/urdf/dh_ag95_controlled.urdf.xacro (robot description, xacro)
@@ -1,5 +1,7 @@
 <?xml version="1.0"?>
 <robot name="dh_ag95_controlled" xmlns:xacro="http://www.ros.org/wiki/xacro">
-  <xacro:arg name="prefix" default="dh_ag95"/>
+  <xacro:arg name="prefix" default=""/>
+  <xacro:arg name="use_mesh" default="true"/>
+  <xacro:arg name="hardware_name" default="dh_ag95_hardware"/>
   <xacro:arg name="transport_type" default="official_serial"/>
   <xacro:arg name="port" default="/dev/ttyACM0"/>
@@ -11,14 +13,23 @@
   <xacro:arg name="gripper_id" default="1"/>
   <xacro:arg name="command_unit" default="normalized"/>
-  <link name="world"/>
+  <xacro:arg name="stroke_m" default="0.095"/>
+  <xacro:arg name="default_force_percent" default="30"/>
+  <xacro:arg name="auto_initialize" default="true"/>
   <xacro:include filename="$(find dh_ag95_description)/urdf/dh_ag95_macro.urdf.xacro"/>
   <xacro:include filename="$(find dh_ag95_description)/urdf/dh_ag95.ros2_control.xacro"/>
-  <xacro:dh_ag95_gripper prefix="$(arg prefix)" parent="world">
+  <link name="world"/>
+  <link name="$(arg prefix)ag95_mount_link"/>
+  <joint name="$(arg prefix)world_to_ag95_mount" type="fixed">
+    <parent link="world"/>
+    <child link="$(arg prefix)ag95_mount_link"/>
+    <origin xyz="0 0 0" rpy="0 0 0"/>
+  </joint>
+  <xacro:dh_ag95_gripper prefix="$(arg prefix)" parent="$(arg prefix)ag95_mount_link" use_mesh="$(arg use_mesh)">
     <origin xyz="0 0 0" rpy="0 0 0"/>
   </xacro:dh_ag95_gripper>
   <xacro:dh_ag95_ros2_control
-    name="$(arg prefix)"
+    name="$(arg hardware_name)"
     prefix="$(arg prefix)"
-    gripper_id="$(arg gripper_id)"
+    plugin="dh_ag95_controllers/DhAg95Hardware"
     transport_type="$(arg transport_type)"
     port="$(arg port)"
@@ -28,4 +39,8 @@
     pcan_channel="$(arg pcan_channel)"
     pcan_bitrate="$(arg pcan_bitrate)"
-    command_unit="$(arg command_unit)"/>
+    gripper_id="$(arg gripper_id)"
+    command_unit="$(arg command_unit)"
+    stroke_m="$(arg stroke_m)"
+    default_force_percent="$(arg default_force_percent)"
+    auto_initialize="$(arg auto_initialize)"/>
 </robot>

File: src/dh_ag95_description/urdf/dh_ag95_macro.urdf.xacro (robot description, xacro)
@@ -1,75 +1,250 @@
 <?xml version="1.0"?>
 <robot xmlns:xacro="http://www.ros.org/wiki/xacro">
-  <!-- Pure visual/collision/kinematic description macro, no ros2_control tags. -->
-  <xacro:macro name="dh_ag95_gripper" params="prefix:=dh_ag95 parent:=world *origin">
-    <link name="${prefix}_base_link">
-      <visual>
-        <origin xyz="0 0 0.025" rpy="0 0 0"/>
-        <geometry><box size="0.085 0.045 0.05"/></geometry>
-        <material name="${prefix}_dark_gray"><color rgba="0.15 0.15 0.15 1"/></material>
-      </visual>
-      <collision>
-        <origin xyz="0 0 0.025" rpy="0 0 0"/>
-        <geometry><box size="0.085 0.045 0.05"/></geometry>
-      </collision>
-      <inertial>
-        <origin xyz="0 0 0.025" rpy="0 0 0"/>
-        <mass value="1.0"/>
-        <inertia ixx="0.001" ixy="0" ixz="0" iyy="0.001" iyz="0" izz="0.001"/>
-      </inertial>
-    </link>
-    <joint name="${prefix}_mount_joint" type="fixed">
+  <!--
+    DH-Robotics AG-95 description macro.
+    This file reorganizes the public DH-Robotics AG-95 ROS1 description into a ROS2-friendly xacro macro.
+    Main kinematic values, joint names, mimic multipliers, inertial values and mesh filenames are taken
+    from the official dh_robotics_ag95_description xacro.
+  -->
+  <xacro:macro name="dh_ag95_gripper" params="
+    prefix
+    parent
+    *origin">
+    <material name="${prefix}dh_ag95_gripper_black_material" >
+      <color rgba="0.15 0.15 0.15 1.0"/>
+    </material>
+    <material name="${prefix}dh_ag95_gripper_white_material" >
+      <color rgba="0.85 0.85 0.85 1.0"/>
+    </material>
+    <joint name="${prefix}gripper_base_joint" type="fixed">
       <parent link="${parent}"/>
-      <child link="${prefix}_base_link"/>
+      <child link="${prefix}gripper_base_link"/>
       <xacro:insert_block name="origin"/>
     </joint>
-    <link name="${prefix}_left_finger_link">
-      <visual>
-        <origin xyz="0 0.0275 0.085" rpy="0 0 0"/>
-        <geometry><box size="0.018 0.018 0.07"/></geometry>
-        <material name="${prefix}_silver"><color rgba="0.75 0.75 0.75 1"/></material>
-      </visual>
-      <collision>
-        <origin xyz="0 0.0275 0.085" rpy="0 0 0"/>
-        <geometry><box size="0.018 0.018 0.07"/></geometry>
-      </collision>
-      <inertial>
-        <origin xyz="0 0.0275 0.085" rpy="0 0 0"/>
-        <mass value="0.15"/>
-        <inertia ixx="0.0001" ixy="0" ixz="0" iyy="0.0001" iyz="0" izz="0.0001"/>
-      </inertial>
-    </link>
-    <link name="${prefix}_right_finger_link">
-      <visual>
-        <origin xyz="0 -0.0275 0.085" rpy="0 0 0"/>
-        <geometry><box size="0.018 0.018 0.07"/></geometry>
-        <material name="${prefix}_silver"/>
-      </visual>
-      <collision>
-        <origin xyz="0 -0.0275 0.085" rpy="0 0 0"/>
-        <geometry><box size="0.018 0.018 0.07"/></geometry>
-      </collision>
-      <inertial>
-        <origin xyz="0 -0.0275 0.085" rpy="0 0 0"/>
-        <mass value="0.15"/>
-        <inertia ixx="0.0001" ixy="0" ixz="0" iyy="0.0001" iyz="0" izz="0.0001"/>
-      </inertial>
-    </link>
-    <!-- Normalized opening joint: 0.0=open, 1.0=closed by default in the driver mapping. -->
-    <joint name="${prefix}_finger_joint" type="prismatic">
-      <parent link="${prefix}_base_link"/>
-      <child link="${prefix}_left_finger_link"/>
-      <origin xyz="0 0 0" rpy="0 0 0"/>
-      <axis xyz="0 -1 0"/>
-      <limit lower="0.0" upper="1.0" effort="100" velocity="1.0"/>
-    </joint>
-    <joint name="${prefix}_right_finger_mimic_joint" type="prismatic">
-      <parent link="${prefix}_base_link"/>
-      <child link="${prefix}_right_finger_link"/>
-      <origin xyz="0 0 0" rpy="0 0 0"/>
+    <link name="${prefix}gripper_base_link">
+      <visual>
+        <geometry>
+          <mesh filename="package://dh_ag95_description/meshes/visual/base_link.STL" scale="0.001 0.001 0.001"/>
+        </geometry>
+        <material name="${prefix}dh_ag95_gripper_black_material"/>
+      </visual>
+      <collision>
+        <geometry>
+          <mesh filename="package://dh_ag95_description/meshes/visual/base_link.STL" scale="0.001 0.001 0.001"/>
+        </geometry>
+      </collision>
+      <inertial>
+        <mass value="0.83416"/>
+        <origin xyz="0 0 0"/>
+        <inertia ixx="0.0013016" ixy="-6.9374e-07" ixz="5.9848e-07" iyy="0.00049972" iyz="2.0244e-07" izz="0.001498"/>
+      </inertial>
+    </link>
+    <joint name="${prefix}gripper_finger1_joint" type="revolute">
+      <parent link="${prefix}gripper_base_link"/>
+      <child link="${prefix}gripper_finger1_knuckle_link"/>
+      <axis xyz="0 -1 0"/>
+      <origin rpy="0 0 ${pi}" xyz="-0.016 0 0.10586"/>
+      <limit lower="0.0" upper="0.65" velocity="2.0" effort="1000"/>
+    </joint>
+    <joint name="${prefix}gripper_finger2_joint" type="revolute">
+      <parent link="${prefix}gripper_base_link"/>
+      <child link="${prefix}gripper_finger2_knuckle_link"/>
+      <axis xyz="0 -1 0"/>
+      <origin rpy="0 0 0" xyz="0.016 0 0.10586"/>
+      <limit lower="-3.14" upper="3.14" velocity="100.0" effort="1000"/>
+      <mimic joint="${prefix}gripper_finger1_joint" multiplier="1.0" offset="0.0"/>
+    </joint>
+    <link name="${prefix}gripper_finger1_knuckle_link">
+      <visual>
+        <geometry>
+          <mesh filename="package://dh_ag95_description/meshes/visual/crank_Link.STL" scale="0.001 0.001 0.001"/>
+        </geometry>
+        <material name="${prefix}dh_ag95_gripper_white_material"/>
+      </visual>
+      <collision>
+        <geometry>
+          <mesh filename="package://dh_ag95_description/meshes/visual/crank_Link.STL" scale="0.001 0.001 0.001"/>
+        </geometry>
+      </collision>
+      <inertial>
+        <mass value="0.011111"/>
+        <origin xyz="0 0 0"/>
+        <inertia ixx="3.88172e-06" ixy="-2.29456e-13" ixz="8.33e-07" iyy="1.92174e-06" iyz="2.04435e-13" izz="4.32374e-06"/>
+      </inertial>
+    </link>
+    <link name="${prefix}gripper_finger2_knuckle_link">
+      <visual>
+        <geometry>
+          <mesh filename="package://dh_ag95_description/meshes/visual/crank_Link.STL" scale="0.001 0.001 0.001"/>
+        </geometry>
+        <material name="${prefix}dh_ag95_gripper_white_material"/>
+      </visual>
+      <collision>
+        <geometry>
+          <mesh filename="package://dh_ag95_description/meshes/visual/crank_Link.STL" scale="0.001 0.001 0.001"/>
+        </geometry>
+      </collision>
+      <inertial>
+        <mass value="0.011111"/>
+        <origin xyz="0 0 0"/>
+        <inertia ixx="3.88172e-06" ixy="-2.29456e-13" ixz="8.33e-07" iyy="1.92174e-06" iyz="2.04435e-13" izz="4.32374e-06"/>
+      </inertial>
+    </link>
+    <joint name="${prefix}gripper_finger1_finger_joint" type="continuous">
+      <parent link="${prefix}gripper_finger1_knuckle_link"/>
+      <child link="${prefix}gripper_finger1_finger_link"/>
+      <axis xyz="0 -1 0"/>
+      <origin xyz="0.0292080077784 0 -0.0227132622407" rpy="0 0 0"/>
+      <limit lower="-3.14" upper="3.14" velocity="100.0" effort="0.1"/>
+      <mimic joint="${prefix}gripper_finger1_joint" multiplier="0.4563942" offset="0"/>
+    </joint>
+    <joint name="${prefix}gripper_finger2_finger_joint" type="continuous">
+      <parent link="${prefix}gripper_finger2_knuckle_link"/>
+      <child link="${prefix}gripper_finger2_finger_link"/>
+      <axis xyz="0 -1 0"/>
+      <origin xyz="0.0292080077784 0 -0.0227132622407" rpy="0 0 0"/>
+      <limit lower="-3.14" upper="3.14" velocity="100.0" effort="0.1"/>
+      <mimic joint="${prefix}gripper_finger1_joint" multiplier="0.4563942" offset="0"/>
+    </joint>
+    <link name="${prefix}gripper_finger1_finger_link">
+      <visual>
+        <geometry>
+          <mesh filename="package://dh_ag95_description/meshes/visual/rod_Link.STL" scale="0.001 0.001 0.001"/>
+        </geometry>
+        <material name="${prefix}dh_ag95_gripper_black_material"/>
+      </visual>
+      <collision>
+        <geometry>
+          <mesh filename="package://dh_ag95_description/meshes/visual/rod_Link.STL" scale="0.001 0.001 0.001"/>
+        </geometry>
+      </collision>
+      <inertial>
+        <mass value="0.0222871"/>
+        <origin xyz="0 0 0"/>
+        <inertia ixx="8.72836e-06" ixy="7.0843e-15" ixz="-2.18833e-06" iyy="7.26157e-06" iyz="7.6579e-15" izz="3.3425e-06"/>
+      </inertial>
+    </link>
+    <link name="${prefix}gripper_finger2_finger_link">
+      <visual>
+        <geometry>
+          <mesh filename="package://dh_ag95_description/meshes/visual/rod_Link.STL" scale="0.001 0.001 0.001"/>
+        </geometry>
+        <material name="${prefix}dh_ag95_gripper_black_material"/>
+      </visual>
+      <collision>
+        <geometry>
+          <mesh filename="package://dh_ag95_description/meshes/visual/rod_Link.STL" scale="0.001 0.001 0.001"/>
+        </geometry>
+      </collision>
+      <inertial>
+        <mass value="0.0222871"/>
+        <origin xyz="0 0 0"/>
+        <inertia ixx="8.72836e-06" ixy="7.0843e-15" ixz="-2.18833e-06" iyy="7.26157e-06" iyz="7.6579e-15" izz="3.3425e-06"/>
+      </inertial>
+    </link>
+    <joint name="${prefix}gripper_finger1_inner_knuckle_joint" type="continuous">
+      <parent link="${prefix}gripper_base_link"/>
+      <child link="${prefix}gripper_finger1_inner_knuckle_link"/>
+      <axis xyz="0 -1 0"/>
+      <origin rpy="0 0 ${pi}" xyz="-0.016 0 0.10586"/>
+      <limit lower="-3.14" upper="3.14" velocity="100.0" effort="0.1"/>
+      <mimic joint="${prefix}gripper_finger1_joint" multiplier="1.49462955" offset="0"/>
+    </joint>
+    <joint name="${prefix}gripper_finger2_inner_knuckle_joint" type="continuous">
+      <parent link="${prefix}gripper_base_link"/>
+      <child link="${prefix}gripper_finger2_inner_knuckle_link"/>
+      <axis xyz="0 -1 0"/>
+      <origin rpy="0 0 0" xyz="0.016 0 0.10586"/>
+      <limit lower="-3.14" upper="3.14" velocity="100.0" effort="0.1"/>
+      <mimic joint="${prefix}gripper_finger1_joint" multiplier="1.49462955" offset="0"/>
+    </joint>
+    <link name="${prefix}gripper_finger1_inner_knuckle_link">
+      <visual>
+        <geometry>
+          <mesh filename="package://dh_ag95_description/meshes/visual/proximal_phalanx_Link.STL" scale="0.001 0.001 0.001"/>
+        </geometry>
+        <material name="${prefix}dh_ag95_gripper_black_material"/>
+      </visual>
+      <collision>
+        <geometry>
+          <mesh filename="package://dh_ag95_description/meshes/visual/proximal_phalanx_Link.STL" scale="0.001 0.001 0.001"/>
+        </geometry>
+      </collision>
+      <inertial>
+        <mass value="0.0318004"/>
+        <origin xyz="0 0 0"/>
+        <inertia ixx="1.39848e-05" ixy="-9.54763e-15" ixz="-5.01422e-06" iyy="1.04943e-05" iyz="8.94585e-16" izz="1.36183e-05"/>
+      </inertial>
+    </link>
+    <link name="${prefix}gripper_finger2_inner_knuckle_link">
+      <visual>
+        <geometry>
+          <mesh filename="package://dh_ag95_description/meshes/visual/proximal_phalanx_Link.STL" scale="0.001 0.001 0.001"/>
+        </geometry>
+        <material name="${prefix}dh_ag95_gripper_black_material"/>
+      </visual>
+      <collision>
+        <geometry>
+          <mesh filename="package://dh_ag95_description/meshes/visual/proximal_phalanx_Link.STL" scale="0.001 0.001 0.001"/>
+        </geometry>
+      </collision>
+      <inertial>
+        <mass value="0.0318004"/>
+        <origin xyz="0 0 0"/>
+        <inertia ixx="1.39848e-05" ixy="-9.54763e-15" ixz="-5.01422e-06" iyy="1.04943e-05" iyz="8.94585e-16" izz="1.36183e-05"/>
+      </inertial>
+    </link>
+    <joint name="${prefix}gripper_finger1_finger_tip_joint" type="continuous">
+      <parent link="${prefix}gripper_finger1_inner_knuckle_link"/>
+      <child link="${prefix}gripper_finger1_finger_tip_link"/>
       <axis xyz="0 1 0"/>
-      <limit lower="0.0" upper="1.0" effort="100" velocity="1.0"/>
-      <mimic joint="${prefix}_finger_joint" multiplier="1.0" offset="0.0"/>
-    </joint>
+      <origin xyz="0.0394969463769 0 0.0382752038125" rpy="0 0 0"/>
+      <limit lower="-3.14" upper="3.14" velocity="100.0" effort="0.1"/>
+      <mimic joint="${prefix}gripper_finger1_joint" multiplier="1.49462955" offset="0"/>
+    </joint>
+    <joint name="${prefix}gripper_finger2_finger_tip_joint" type="continuous">
+      <parent link="${prefix}gripper_finger2_inner_knuckle_link"/>
+      <child link="${prefix}gripper_finger2_finger_tip_link"/>
+      <axis xyz="0 1 0"/>
+      <origin xyz="0.0394969463769 0 0.0382752038125" rpy="0 0 0"/>
+      <limit lower="-3.14" upper="3.14" velocity="100.0" effort="0.1"/>
+      <mimic joint="${prefix}gripper_finger1_joint" multiplier="1.49462955" offset="0"/>
+    </joint>
+    <link name="${prefix}gripper_finger1_finger_tip_link">
+      <visual>
+        <geometry>
+          <mesh filename="package://dh_ag95_description/meshes/visual/distal_phalanx_Link.STL" scale="0.001 0.001 0.001"/>
+        </geometry>
+        <material name="${prefix}dh_ag95_gripper_white_material"/>
+      </visual>
+      <collision>
+        <geometry>
+          <mesh filename="package://dh_ag95_description/meshes/visual/distal_phalanx_Link.STL" scale="0.001 0.001 0.001"/>
+        </geometry>
+      </collision>
+      <inertial>
+        <mass value="0.0124305"/>
+        <origin xyz="0 0 0"/>
+        <inertia ixx="2.84217e-06" ixy="-2.48048e-15" ixz="8.24539e-07" iyy="3.03961e-06" iyz="2.16427e-13" izz="1.11815e-06"/>
+      </inertial>
+    </link>
+    <link name="${prefix}gripper_finger2_finger_tip_link">
+      <visual>
+        <geometry>
+          <mesh filename="package://dh_ag95_description/meshes/visual/distal_phalanx_Link.STL" scale="0.001 0.001 0.001"/>
+        </geometry>
+        <material name="${prefix}dh_ag95_gripper_white_material"/>
+      </visual>
+      <collision>
+        <geometry>
+          <mesh filename="package://dh_ag95_description/meshes/visual/distal_phalanx_Link.STL" scale="0.001 0.001 0.001"/>
+        </geometry>
+      </collision>
+      <inertial>
+        <mass value="0.0124305"/>
+        <origin xyz="0 0 0"/>
+        <inertia ixx="2.84217e-06" ixy="-2.48048e-15" ixz="8.24539e-07" iyy="3.03961e-06" iyz="2.16427e-13" izz="1.11815e-06"/>
+      </inertial>
+    </link>
   </xacro:macro>
 </robot>
