Commit message: fxied ros2 controller

File: src/dh_ag95_description/urdf/dh_ag95.ros2_control.xacro (robot description, xacro)
@@ -1,10 +1,27 @@
 <?xml version="1.0"?>
 <robot xmlns:xacro="http://www.ros.org/wiki/xacro">
+  <!--
+  本文件支持多种传输类型，包括官方串口、CAN串口、Socket CAN（Linux）、PCAN（Windows）等。
+  你可以通过 'transport_type' 参数选择不同的协议（official_serial、slcan、socketcan、pcanbasic、modbus_rtu(暂不支持)）
+  official_serial 的参数包括： port（串口号）、baudrate（波特率）；
+  slcan 的参数包括： port（串口号）、baudrate（波特率）、can_bitrate（CAN波特率）；
+  socketcan 的参数包括： can_interface（CAN接口）、can_bitrate（CAN波特率）；
+  pcanbasic 的参数包括： pcan_channel（PCAN通道）、pcan_bitrate（PCAN波特率）；
+  -->
+  <!--
+  This module supports various transport types, including official serial, slcan, SocketCAN (Linux), and PCAN (Windows).
+  You can select different protocols using the 'transport_type' parameter (options: official_serial, slcan, socketcan, pcanbasic, modbus_rtu [not currently supported]).
+  Parameters for 'official_serial' include: port, baudrate;
+  Parameters for 'slcan' include: port, baudrate, can_bitrate;
+  Parameters for 'socketcan' include: can_interface, can_bitrate;
+  Parameters for 'pcanbasic' include: pcan_channel, pcan_bitrate;
+  -->
   <xacro:macro name="dh_ag95_ros2_control" params="
+      prefix
       name:=dh_ag95_hardware
-      prefix:=
+      use_fake_hardware:=false
       transport_type:=official_serial
-      port:=/dev/ttyACM0
-      baudrate:=115200
+      serial_port:=/dev/ttyACM0
+      serial_baudrate:=115200
       can_interface:=can0
       can_bitrate:=500000
@@ -15,35 +32,68 @@
       stroke_m:=0.095
       default_force_percent:=30
-      auto_initialize:=true">
-    <ros2_control name="${name}" type="actuator">
-      <hardware>
-        <plugin>dh_ag95_controllers/DhAg95Hardware</plugin>
-        <param name="transport_type">${transport_type}</param>
-        <param name="port">${port}</param>
-        <param name="baudrate">${baudrate}</param>
-        <param name="can_interface">${can_interface}</param>
-        <param name="can_bitrate">${can_bitrate}</param>
-        <param name="pcan_channel">${pcan_channel}</param>
-        <param name="pcan_bitrate">${pcan_bitrate}</param>
-        <param name="gripper_id">${gripper_id}</param>
-        <param name="command_unit">${command_unit}</param>
-        <param name="stroke_m">${stroke_m}</param>
-        <param name="default_force_percent">${default_force_percent}</param>
-        <param name="auto_initialize">${auto_initialize}</param>
-      </hardware>
-      <joint name="${prefix}gripper_finger1_joint">
-        <command_interface name="position">
-          <param name="min">0.0</param>
-          <param name="max">1.0</param>
-        </command_interface>
-        <command_interface name="effort">
-          <param name="min">20.0</param>
-          <param name="max">100.0</param>
-        </command_interface>
-        <state_interface name="position"/>
-        <state_interface name="velocity"/>
-        <state_interface name="effort"/>
-      </joint>
-    </ros2_control>
+      auto_initialize:=true
+      rw_rate:=50">
+    <xacro:if value="${use_fake_hardware}">
+      <ros2_control name="${name}" type="system">
+        <hardware>
+          <plugin>mock_components/GenericSystem</plugin>
+          <param name="fake_sensor_commands">false</param>
+          <param name="state_interface_names">
+            <value>position</value>
+            <value>velocity</value>
+            <value>effort</value>
+          </param>
+          <param name="command_interface_names">
+            <value>position</value>
+            <value>effort</value>
+          </param>
+        </hardware>
+        <joint name="${prefix}gripper_finger1_joint">
+          <command_interface name="position">
+            <param name="min">0.0</param>
+            <param name="max">1.0</param>
+          </command_interface>
+          <command_interface name="effort">
+            <param name="min">20.0</param>
+            <param name="max">100.0</param>
+          </command_interface>
+          <state_interface name="position"/>
+          <state_interface name="velocity"/>
+          <state_interface name="effort"/>
+        </joint>
+      </ros2_control>
+    </xacro:if>
+    <xacro:unless value="${use_fake_hardware}">
+      <ros2_control name="${name}" type="actuator">
+        <hardware>
+          <plugin>dh_ag95_controllers/DhAg95Hardware</plugin>
+          <param name="transport_type">${transport_type}</param>
+          <param name="port">${port}</param>
+          <param name="baudrate">${baudrate}</param>
+          <param name="can_interface">${can_interface}</param>
+          <param name="can_bitrate">${can_bitrate}</param>
+          <param name="pcan_channel">${pcan_channel}</param>
+          <param name="pcan_bitrate">${pcan_bitrate}</param>
+          <param name="gripper_id">${gripper_id}</param>
+          <param name="command_unit">${command_unit}</param>
+          <param name="stroke_m">${stroke_m}</param>
+          <param name="default_force_percent">${default_force_percent}</param>
+          <param name="auto_initialize">${auto_initialize}</param>
+        </hardware>
+        <joint name="${prefix}gripper_finger1_joint">
+          <command_interface name="position">
+            <param name="min">0.0</param>
+            <param name="max">1.0</param>
+          </command_interface>
+          <command_interface name="effort">
+            <param name="min">20.0</param>
+            <param name="max">100.0</param>
+          </command_interface>
+          <state_interface name="position"/>
+          <state_interface name="velocity"/>
+          <state_interface name="effort"/>
+        </joint>
+      </ros2_control>
+    </xacro:unless>
   </xacro:macro>
 </robot>

File: src/dh_ag95_description/urdf/dh_ag95_controlled.urdf.xacro (robot description, xacro)
@@ -2,9 +2,8 @@
 <robot name="dh_ag95_controlled" xmlns:xacro="http://www.ros.org/wiki/xacro">
   <xacro:arg name="prefix" default=""/>
-  <xacro:arg name="use_mesh" default="true"/>
   <xacro:arg name="hardware_name" default="dh_ag95_hardware"/>
   <xacro:arg name="transport_type" default="official_serial"/>
-  <xacro:arg name="port" default="/dev/ttyACM0"/>
-  <xacro:arg name="baudrate" default="115200"/>
+  <xacro:arg name="serial_port" default="/dev/ttyACM0"/>
+  <xacro:arg name="serial_baudrate" default="115200"/>
   <xacro:arg name="can_interface" default="can0"/>
   <xacro:arg name="can_bitrate" default="500000"/>
@@ -16,4 +15,6 @@
   <xacro:arg name="default_force_percent" default="30"/>
   <xacro:arg name="auto_initialize" default="true"/>
+  <xacro:arg name="use_fake_hardware" default="false"/>
+  <xacro:arg name="rw_rate" default="50"/>
   <xacro:include filename="$(find dh_ag95_description)/urdf/dh_ag95_macro.urdf.xacro"/>
   <xacro:include filename="$(find dh_ag95_description)/urdf/dh_ag95.ros2_control.xacro"/>
@@ -25,14 +26,14 @@
     <origin xyz="0 0 0" rpy="0 0 0"/>
   </joint>
-  <xacro:dh_ag95_gripper prefix="$(arg prefix)" parent="$(arg prefix)ag95_mount_link" use_mesh="$(arg use_mesh)">
+  <xacro:dh_ag95_gripper prefix="$(arg prefix)" parent="$(arg prefix)ag95_mount_link">
     <origin xyz="0 0 0" rpy="0 0 0"/>
   </xacro:dh_ag95_gripper>
   <xacro:dh_ag95_ros2_control
+    prefix="$(arg prefix)"
     name="$(arg hardware_name)"
-    prefix="$(arg prefix)"
-    plugin="dh_ag95_controllers/DhAg95Hardware"
+    use_fake_hardware="$(arg use_fake_hardware)"
     transport_type="$(arg transport_type)"
-    port="$(arg port)"
-    baudrate="$(arg baudrate)"
+    serial_port="$(arg serial_port)"
+    serial_baudrate="$(arg serial_baudrate)"
     can_interface="$(arg can_interface)"
     can_bitrate="$(arg can_bitrate)"
@@ -43,4 +44,5 @@
     stroke_m="$(arg stroke_m)"
     default_force_percent="$(arg default_force_percent)"
-    auto_initialize="$(arg auto_initialize)"/>
+    auto_initialize="$(arg auto_initialize)"
+    rw_rate="$(arg rw_rate)"/>
 </robot>
